File: thermostat_master.kicad_pcb (KiCad board)
At the start: 2 copper layers, 96 x 63 mm, 11 parts, among them J1 Conn_01x14, J2 Conn_01x04, J3 Conn_01x04, J4 Conn_01x02, J5 Screw_Terminal_01x02, K1 G3MB202PDC12, U1 esp32_38_pins

Commit message: v1.1 PCB
Other:
- board text added: "3.3V"
- board text added: "GPIO10"
- board text added: "GPIO11"
- board text added: "GPIO12"
- board text added: "GPIO14"
- board text added: "GPIO25"
- board text added: "GPIO26"
- board text added: "GPIO27"
- board text added: "GPIO32"
- board text added: "GPIO33"
- board text added: "GPIO34"
- board text added: "GPIO35"
- board text added: "GPIO36"
- board text added: "GPIO39"
- board text added: "GPIO9"
- board text added: "RST/EN"
- board text added: "VIN 5V"
Changed lines of the file:
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@@
   (general
     (thickness 1.6)
-    (drawings 41)
+    (drawings 60)
     (tracks 118)
     (zones 0)
@@
   (page A4)
   (layers
-    (0 F.Cu signal)
-    (31 B.Cu mixed)
+    (0 F.Cu signal hide)
+    (31 B.Cu mixed hide)
     (33 F.Adhes user)
     (35 F.Paste user)
@@
     (44 Edge.Cuts user)
     (45 Margin user)
-    (46 B.CrtYd user)
+    (46 B.CrtYd user hide)
     (47 F.CrtYd user)
     (49 F.Fab user hide)
@@
   (module My_Libraries:ESP32_Keeyes_38_Pins (layer F.Cu)
     (at 153.67 80.264)
-    (fp_text reference U1 (at 14.8082 0.0254 180) (layer F.SilkS)
+    (fp_text reference U1 (at 0.254 0 180) (layer F.SilkS)
       (effects (font (size 1 1) (thickness 0.15)))
     )
@@
     )
   )
+  (gr_text "VIN 5V" (at 137.668 103.124) (layer F.SilkS)
+    (effects (font (size 1 1) (thickness 0.15)))
+  )
+  (gr_text GPIO11 (at 137.414 100.584) (layer F.SilkS)
+    (effects (font (size 1 1) (thickness 0.15)))
+  )
+  (gr_text GPIO10 (at 137.414 98.044) (layer F.SilkS)
+    (effects (font (size 1 1) (thickness 0.15)))
+  )
+  (gr_text GPIO9 (at 137.922 95.504) (layer F.SilkS)
+    (effects (font (size 1 1) (thickness 0.15)))
+  )
+  (gr_text GPIO12 (at 137.414 92.964) (layer F.SilkS)
+    (effects (font (size 1 1) (thickness 0.15)))
+  )
+  (gr_text GND (at 138.684 90.424) (layer F.SilkS)
+    (effects (font (size 1 1) (thickness 0.15)))
+  )
+  (gr_text GPIO12 (at 137.414 87.884) (layer F.SilkS)
+    (effects (font (size 1 1) (thickness 0.15)))
+  )
+  (gr_text GPIO14 (at 137.414 85.344) (layer F.SilkS)
+    (effects (font (size 1 1) (thickness 0.15)))
+  )
+  (gr_text GPIO27 (at 137.414 82.804) (layer F.SilkS)
+    (effects (font (size 1 1) (thickness 0.15)))
+  )
+  (gr_text GPIO26 (at 137.414 80.264) (layer F.SilkS)
+    (effects (font (size 1 1) (thickness 0.15)))
+  )
+  (gr_text GPIO25 (at 137.414 77.724) (layer F.SilkS)
+    (effects (font (size 1 1) (thickness 0.15)))
+  )
+  (gr_text GPIO33 (at 137.414 75.184) (layer F.SilkS)
+    (effects (font (size 1 1) (thickness 0.15)))
+  )
+  (gr_text GPIO32 (at 137.414 72.644) (layer F.SilkS)
+    (effects (font (size 1 1) (thickness 0.15)))
+  )
+  (gr_text GPIO35 (at 137.414 70.104) (layer F.SilkS)
+    (effects (font (size 1 1) (thickness 0.15)))
+  )
+  (gr_text GPIO34 (at 137.414 67.564) (layer F.SilkS)
+    (effects (font (size 1 1) (thickness 0.15)))
+  )
+  (gr_text GPIO39 (at 137.414 65.024) (layer F.SilkS)
+    (effects (font (size 1 1) (thickness 0.15)))
+  )
+  (gr_text GPIO36 (at 137.414 62.484) (layer F.SilkS)
+    (effects (font (size 1 1) (thickness 0.15)))
+  )
+  (gr_text RST/EN (at 137.414 59.944) (layer F.SilkS)
+    (effects (font (size 1 1) (thickness 0.15)))
+  )
+  (gr_text 3.3V (at 138.43 57.404) (layer F.SilkS)
+    (effects (font (size 1 1) (thickness 0.15)))
+  )
   (gr_text v1.1 (at 177.8508 50.3936) (layer F.SilkS)
